File: pcbshizz/weatherstation.kicad_sch (KiCad schematic)
At the start: 24 parts, among them U2 ESD7104MUTAG, U3 ESP32-S3-MINI-1-N8, U4 ENS210, U5 TLV75801PDRV

Commit message: ho gya funny?
Parts:
- removed U4: ENS210, Package_DFN_QFN:AMS_QFN-4-1EP_2x2mm_P0.95mm_EP0.7x1.6mm, symbol Sensor_Humidity:ENS210
- added J1: Conn_01x03_Socket, Connector_PinSocket_2.54mm:PinSocket_1x03_P2.54mm_Vertical, symbol Connector:Conn_01x03_Socket
- added J2: ~, Connector_PinHeader_2.54mm:PinHeader_1x22_P2.54mm_Vertical, symbol Connector:Conn_01x22_Pin
- added J3: Conn_01x21_Pin, Connector_PinSocket_2.54mm:PinSocket_1x21_P2.54mm_Vertical, symbol Connector:Conn_01x21_Pin
- added U1: MS860702BA01-50, MS860702BA01-50:TE_MS860702BA01-50, symbol MS860702BA01-50:MS860702BA01-50
- U3: footprint ESP32-S3-MINI-1-N8:XCVR_ESP32-S3-MINI-1-N8 -> RF_Module:ESP32-S2-MINI-1
Connections:
- net 3V3: now also J1.3 (Pin_3), J2.1 (Pin_1), U1.1 (VDD)
- net 5VUSB: now also J2.21 (Pin_21)
- net ESP32_EN: now also J3.2 (Pin_2)
- net GND: now also J1.1 (Pin_1), J2.22 (Pin_22), J3.1 (Pin_1), U1.3 (GND)
- net GPIO0: now also J2.2 (Pin_2)
- net GPIO1: now also J2.3 (Pin_3)
- net GPIO10: now also J2.12 (Pin_12)
- net GPIO11: now also J2.13 (Pin_13)
- net GPIO12: now also J2.14 (Pin_14)
- net GPIO13: now also J2.15 (Pin_15)
- net GPIO14: now also J2.16 (Pin_16)
- net GPIO15: now also J2.17 (Pin_17)
- net GPIO16: now also J2.18 (Pin_18)
- net GPIO2: now also J2.4 (Pin_4)
- net GPIO21: now also J3.18 (Pin_18)
- net GPIO26: now also J3.17 (Pin_17)
- net GPIO3: now also J2.5 (Pin_5)
- net GPIO33: now also J3.16 (Pin_16)
- net GPIO34: now also J3.15 (Pin_15)
- net GPIO35: now also J3.14 (Pin_14)
- net GPIO36: now also J3.13 (Pin_13)
- net GPIO37: now also J3.12 (Pin_12)
- net GPIO38: now also J3.11 (Pin_11)
- net GPIO39: now also J3.10 (Pin_10)
- net GPIO4: now also J2.6 (Pin_6)
- net GPIO40: now also J3.9 (Pin_9)
- net GPIO41: now also J3.8 (Pin_8)
- net GPIO42: now also J3.7 (Pin_7)
- net GPIO45: now also J3.4 (Pin_4)
- net GPIO46: now also J3.3 (Pin_3)
- net GPIO47: now also J1.2 (Pin_2)
- net GPIO48: now also J3.21 (Pin_21)
- net GPIO5: now also J2.7 (Pin_7)
- net GPIO6: now also J2.8 (Pin_8)
- net GPIO7: now also J2.9 (Pin_9)
- net GPIO8: now also J2.10 (Pin_10)
- net GPIO9: now also J2.11 (Pin_11)
- net I2C_SCL: now also J2.19 (Pin_19), U1.8 (SCL)
- net I2C_SDA: now also J2.20 (Pin_20), U1.7 (SDA)
- net RXD: now also J3.5 (Pin_5)
- net TXD: now also J3.6 (Pin_6)
- no-connect marks 3 -> 5

Commit message: baguette 👍
Parts:
- removed J2: ~, Connector_PinHeader_2.54mm:PinHeader_1x22_P2.54mm_Vertical, symbol Connector:Conn_01x22_Pin
- removed J3: Conn_01x21_Pin, Connector_PinSocket_2.54mm:PinSocket_1x21_P2.54mm_Vertical, symbol Connector:Conn_01x21_Pin
- added J2: Conn_01x02_Pin, Connector_PinSocket_2.54mm:PinSocket_1x02_P2.54mm_Vertical, symbol Connector:Conn_01x02_Pin
Connections:
- net I2C_SCL: now also J2.1 (Pin_1)
- net I2C_SDA: now also J2.2 (Pin_2)
- no-connect marks 5 -> 3
