File: pcbshizz/weatherstation.kicad_pcb (KiCad board)
At the start: 2 copper layers, 24 parts, among them U1 ESP32-S3-MINI-1, U2 ESD7104MUTAG, U4 ENS210, U5 TLV75801PDRV

Commit message: ho gya funny?
Parts:
- added J1: Conn_01x03_Socket, Connector_PinSocket_2.54mm:PinSocket_1x03_P2.54mm_Vertical, F.Cu at (78.1, 113.1)
- added J2: ~, Connector_PinHeader_2.54mm:PinHeader_1x22_P2.54mm_Vertical, F.Cu at (90.2, 113.0)
- added J3: Conn_01x21_Pin, Connector_PinSocket_2.54mm:PinSocket_1x21_P2.54mm_Vertical, F.Cu at (92.8, 117.0)
- added U1: MS860702BA01-50, MS860702BA01-50:TE_MS860702BA01-50, F.Cu at (107.9, 107.1)
- moved C1 26.6 mm to (97.0, 91.5)
- moved C2 26.6 mm to (97.0, 94.0)
- moved D1 13.4 mm to (94.9, 99.4)
- moved JUSB1 11.7 mm to (83.7, 88.3)
- moved U2 10.5 mm to (90.1, 88.5)
- moved U1 4.06 mm to (111.8, 88.8)

Commit message: baguette 👍
Parts:
- removed J3: Conn_01x21_Pin, Connector_PinSocket_2.54mm:PinSocket_1x21_P2.54mm_Vertical
- removed the U1 at (111.8, 88.8)
- added U3: ESP32-S3-MINI-1-N8, RF_Module:ESP32-S2-MINI-1, F.Cu at (110.8, 87.2)
- J2: value ~ -> Conn_01x02_Pin; footprint Connector_PinHeader_2.54mm:PinHeader_1x22_P2.54mm_Vertical -> Connector_PinSocket_2.54mm:PinSocket_1x02_P2.54mm_Vertical
- moved J1 19.7 mm to (93.1, 100.3)
- moved D1 18.8 mm to (113.5, 101.5)
- moved C2 10.6 mm to (99.3, 83.6), turned to 90 degrees
- moved C1 9.15 mm to (101.8, 83.7), turned to 90 degrees
- moved J2 9.09 mm to (93.1, 104.4)
- moved U2 8.48 mm to (98.6, 87.6)
- moved JUSB1 8.46 mm to (92.2, 87.7)
Connections:
- J1 pad 1: unconnected-(J1-Pin_1-Pad1) -> GND
- J1 pad 2: unconnected-(J1-Pin_2-Pad2) -> /GPIO47
- J1 pad 3: unconnected-(J1-Pin_3-Pad3) -> /3V3
- J2 pad 1: /3V3 -> /I2C_SCL
- J2 pad 2: /GPIO0 -> /I2C_SDA
Other:
- copper layers 2 -> 4

Commit message: eee
Parts:
- added H4: MountingHole, MountingHole:MountingHole_3.2mm_M3, F.Cu at (108.0, 77.5)
- added H5: MountingHole, MountingHole:MountingHole_3.2mm_M3, F.Cu at (108.0, 101.2)
- moved U5 38.2 mm to (108.8, 85.0), turned to 180 degrees
- moved D2 38.2 mm to (108.5, 92.8), turned to 90 degrees
- moved U1 37.4 mm to (128.0, 75.6)
- moved J1 36.2 mm to (118.4, 74.4), turned to -90 degrees
- moved C2 34.4 mm to (133.4, 78.8)
- moved C1 34.4 mm to (135.8, 78.8)
- moved U4 33.5 mm to (122.9, 75.8), turned to 180 degrees
- moved J2 33.3 mm to (113.4, 78.0)
- moved R5 22.8 mm to (132.0, 75.3), turned to -90 degrees
- moved R7 22.8 mm to (112.2, 83.1), turned to 180 degrees
- moved C4 21.6 mm to (135.8, 75.3), turned to 90 degrees
- moved R1 21.4 mm to (105.9, 82.8)
- moved R4 20.9 mm to (133.8, 75.3), turned to -90 degrees
- moved U3 20.9 mm to (131.7, 89.1), turned to -90 degrees
- moved R2 19.2 mm to (109.0, 82.8), turned to 180 degrees
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Routing:
- net /3V3: track 0.00 -> 94.6 mm, vias 0 -> 4
- net /I2C_SCL: track 0.00 -> 40.4 mm, vias 0 -> 2
- net /I2C_SDA: track 0.00 -> 34.9 mm, vias 0 -> 1
- net /GPIO47: track 0.00 -> 32.8 mm, vias 0 -> 2
- net /5VUSB: track 0.00 -> 25.3 mm
- net /USB_N: track 0.00 -> 16.6 mm
- net /USB_P: track 0.00 -> 16.4 mm
- net Net-(JUSB1-CC1): track 0.00 -> 16.0 mm, vias 0 -> 2
- net Net-(D2-A): track 0.00 -> 13.5 mm, vias 0 -> 2
- net Net-(JUSB1-CC2): track 0.00 -> 11.7 mm, vias 0 -> 2
- net /GPIO0: track 0.00 -> 9.95 mm, vias 0 -> 2
- net Net-(U5-FB): track 0.00 -> 8.42 mm
- net /GPIO48: track 0.00 -> 7.79 mm
- net GND: track 0.03 -> 5.93 mm, vias 0 -> 7
- net /ESP32_EN: track 0.00 -> 3.99 mm
- added copper zone on B.Cu, net GND
- added copper zone on F.Cu, net GND
Other:
- board outline added: 38.3 x 33.5 mm
- board text added: "+ve"
- board text added: "-ve"
- board text added: "HALL EFFECT"
- board text added: "SCL"
- board text added: "SDA"
